File: clutch.kicad_sch (KiCad schematic)
At the start: 51 parts, among them SW1 SYNC SW, SW2 RD CLUTCH TRIP

Commit message: Fix messed up part numbers
Parts:
- added DU1-AL: FUSE, symbol ibm:relay-NO
- READ-CL-MAGNET: renamed from R3; value magnet -> READ CL MAGNET
- renumbered 1-7 to 1-5, 2-8 to 2-4, 2-7 to 2-6, 3-7 to 3-3, 4-6 to 4-1, 4-7 to 4-3, 4-8 to 4-6, C3 to C4, DU4-AU2 to DU4-AU, DU4-BU2 to DU4-BU, NPRO3 to NPRO2, Online/Offline1 to Online/OfflineA, Online/Offline to Online/OfflineB, RD7 to R15, RD32 to RD17, RD34 to RD2, RD28 to RD32, RD30 to RD46, RD8 to RD49, RD29 to RD60, RD35 to RD62, RD33 to RD7, RD31 to RD83
Connections:
- net -20: now also DU1-AL.1
- net at 2-6.3, 4-3.3, RD46.2 (A)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: now also DU1-AL.3
Other:
- note added: "Apparently RC 173 RD JAM indicates READ STOP while RC 168 READ STOP indicates READ STOP, STACKER, FUSE, or JAM."
- note removed: "Apparently RC 173 RD JAM indicates READ STOP while RC 168 READ STOP indicates READ STOP, STACKER, or JAM."
- moved on the sheet: 1-5, 2-4, 2-6, 3-3, 3-6, 4-1, 4-3, 4-6, 4H, 7-4, DU4-AU, DU4-BU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
