File: cl.kicad_sch (KiCad schematic)
At the start: 27 parts

Commit message: Fix messed up part numbers
Parts:
- added 1H, 1P: READ HOPPER, symbol ibm:relay-coil
- added R3: HOPPER CARD LEVER, symbol ibm:card lever
- added RD8: R_US, symbol Device:R_US
- renumbered 12-5 to 12-1, 12-3 to 12-4, 12-4 to 12-5, RC10 to RC12, RC7 to RC8, RC8 to RC9, RD5 to RD19, RD10 to RD56, RD9 to RD57, RL4 to RL1, RL2 to RL3
Connections:
- net -20: now also R3.1
- net at 12-4.2, 13P.1: now also 13-3.3; no longer 13-3.1
- net at 6P.1, RC9.1, RL1.1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: now also 12-1.1, 13-3.1; no longer 12-1.3, 13-3.3
- net at 12P.1, RC9.3: now also 12-1.3; no longer 12-1.1
- new net: 1H.1, R3.3, RD8.1
- new net: 1P.1, RD8.2
Other:
- note added: "The card lever relays are picked when the corresponding card lever detects a card. 155°-185°, 242°-307°"
- note removed: "The card lever relays are picked when the corresponding card lever detects a card. (Subject to timing cams.)"
- moved on the sheet: 12-1, 12-4, 12P, 13-3, 13P, 2P, 3P, 6P, RC9, RD56, RD57, RL1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
