File: reader.kicad_sch (KiCad schematic)
At the start: 53 parts, among them SW3 RDR NPRO

Commit message: Fix messed up part numbers
Parts:
- 9-4: renamed from 2-6; value #1 CL -> MOTOR CONTROL
- R2: renamed from RD24; value R_US -> Variable
- renumbered 1-3 to 1-2, 1-2 to 1-3, 10-3 to 10-2, 10-2 to 10-3, 12-1 to 12-3, 9-3 to 9-1, 9-1 to 9-2, 9-2 to 9-3, C2 to C1, C1 to C2, DU2-AU1 to DU2-AU, DU3-AU2 to DU3-AU, NPRO2 to NPRO3, RC4 to RC1, RC9 to RC2, RC1 to RC3, RC2 to RC4, RC3 to RC7, RD3 to RD11, RD1 to RD21, RD18 to RD24, RD6 to RD4, RD23 to RD40, RD4 to RD41, RD11 to RD42, RD25 to RD44, RD22 to RD5, RD26 to RD6, RL1 to RL10
Connections:
- net at 1-3.3, 8P.1, RD41.2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: no longer C2.1
- net at 10-3.1, 2-2.1, RD24.2 (A): now also 1-2.3, 6-2.2; no longer 1-2.1, 6-2.1
- net at 3-2.3, 9-1.1, RC2.3: now also 1-2.1, 6-2.1; no longer 1-2.3, 6-2.2
- net at RD42.1: now also C2.1
Other:
- note added: "100°-185°, 220°-305°, 340°-65°"
- note added: "102°-147°, 222°-267°, 342°-27°"
- note added: "107°-142°, 227°-262°, 347°-22°"
- note added: "22°-107°, 142°-227°, 262°-347°"
- note added: "272°-342°"
- note added: "Delay on pick if hopper empty"
- note removed: "155°-185°, 242°-307°"
- note removed: "340°-65°, 100°-185°, 220°-305°"
- note removed: "342°-27°, 102°-147°, 222°-267°"
- note removed: "Delay on pick"
- moved on the sheet: 1-2, 6-2, 8H, C2, NPRO3, RD41, RD42, RD5
